Commit message: Corrected wrong name of rplidar_gazebo xacro

File: urdf/rplidar.urdf.xacro (robot description, xacro)
@@ -1,4 +1,4 @@
 <?xml version="1.0"?>
-<robot xmlns:xacro="http://www.ros.org/wiki/xacro">
+<robot name="sensor_rplidar" xmlns:xacro="http://www.ros.org/wiki/xacro">
   <xacro:macro name="sensor_rplidar" params="prefix parent prefix_topic:='front_laser' *origin min_angle:=3.14159 max_angle:=-3.14159">
     <joint name="${prefix}_laser_base_joint" type="fixed">
@@ -35,5 +35,5 @@
     <sensor_rplidar_gazebo/>
   </xacro:macro>
-  <xacro:macro name="${prefix}_sensor_rplidar_gazebo">
+  <xacro:macro name="sensor_rplidar_gazebo">
     <gazebo reference="${prefix}_laser_link">
 			<sensor type="ray" name="${prefix}_rplidar_sensor">
@@ -62,5 +62,5 @@
 				</ray>
 				<plugin name="gazebo_ros_rplidar_controller" filename="libgazebo_ros_laser.so">
-					<topicName>${prefix_topic}/scan</topicName>
+					<topicName>${prefix_topic}/rplidar/scan</topicName>
 					<frameName>/${prefix}_laser_link</frameName>
 				</plugin>

File: urdf/sick_s300.urdf.xacro (robot description, xacro)
@@ -64,5 +64,5 @@
 				</ray>
 				<plugin name="${prefix}_controller" filename="libgazebo_ros_laser.so">
-					<topicName>${prefix_topic}/scan</topicName>
+					<topicName>${prefix_topic}/sick_s300/scan</topicName>
 					<frameName>/${prefix}_link</frameName><!-- if not global (leading /) sets the current namespace as a prefix (/ns/name_laser_link) -->
 				</plugin>
