Commit message: Add rbcar-related sensors

File: urdf/axis.urdf.xacro (robot description, xacro)
@@ -17,5 +17,6 @@
         <origin xyz="0.0 0.0 0.0" rpy="0 0 0"/>
         <mass value="0.1"/>
-        <inertia ixx="0.0004008333" ixy="0" ixz="0" iyy="0.0004008333" iyz="0" izz="0.000426666"/>
+        <origin xyz="0 0 0" rpy="0 0 0"/>
+        <inertia ixx="0.1" ixy="0" ixz="0" iyy="0.1" iyz="0" izz="0.1"/>
       </inertial>
       <visual>
@@ -48,7 +49,7 @@
     <link name="${prefix}_pan_link">
       <inertial>
-        <origin xyz="0.0 0.0 0.0" rpy="0 0 0"/>
         <mass value="0.1"/>
-        <inertia ixx="0.0004008333" ixy="0" ixz="0" iyy="0.0004008333" iyz="0" izz="0.000426666"/>
+        <origin xyz="0 0 0" rpy="0 0 0"/>
+        <inertia ixx="0.1" ixy="0" ixz="0" iyy="0.1" iyz="0" izz="0.1"/>
       </inertial>
     </link>
@@ -73,7 +74,7 @@
     <link name="${prefix}_tilt_link">
       <inertial>
-        <origin xyz="0.0 0.0 0.0" rpy="0 0 0"/>
         <mass value="0.1"/>
-        <inertia ixx="0.0004008333" ixy="0" ixz="0" iyy="0.0004008333" iyz="0" izz="0.000426666"/>
+        <origin xyz="0 0 0" rpy="0 0 0"/>
+        <inertia ixx="0.1" ixy="0" ixz="0" iyy="0.1" iyz="0" izz="0.1"/>
       </inertial>
     </link>

File: urdf/imu.urdf.xacro (robot description, xacro)
@@ -24,5 +24,5 @@
 	        <origin rpy="0 0 0" xyz="0 0 0"/>
 	        <geometry>
-	          <box size=".001 .001 .001"/>
+	          <box size="0.001 0.001 0.001"/>
 	        </geometry>
 	      </collision-->
