Commit message: Update sensors

File: urdf/rubedos_viper.urdf.xacro (robot description, xacro)
@@ -74,5 +74,5 @@
         <origin xyz="0 0 0" rpy="0 0 0"/>
         <geometry>
-          <box size="${rubedos_viper_depth} ${rubedos_viper_height} ${rubedos_viper_width}"/>
+          <box size="${rubedos_viper_depth} ${rubedos_viper_width} ${rubedos_viper_height}"/>
           <!--<mesh filename="package://pointgrey_camera_description/meshes/rubedos_viper.dae"/>-->
         </geometry>

File: urdf/sick_microscan3.urdf.xacro (robot description, xacro)
@@ -40,7 +40,7 @@
 	<xacro:macro name="sensor_sick_microscan3_gazebo">
 		<gazebo reference="${prefix}_link">
-			<sensor type="gpu_ray" name="${prefix}_sensor">
+			<sensor type="ray" name="${prefix}_sensor">
 				<pose>0 0 0 0 0 0</pose>
-				<visualize>false</visualize>
+				<visualize>true</visualize>
 				<update_rate>12.5</update_rate>
 				<ray>
@@ -64,5 +64,5 @@
 					</noise>
 				</ray>
-				<plugin name="${prefix}_controller" filename="libgazebo_ros_gpu_laser.so">
+				<plugin name="${prefix}_controller" filename="libgazebo_ros_laser.so">
 					<topicName>${prefix_topic}/scan</topicName>
 					<frameName>/${prefix}_link</frameName>					<!-- if not global (leading /) sets the current namespace as a prefix (/ns/name_laser_link) -->
